File: pcb/buck.kicad_sch (KiCad schematic)
At the start: 19 parts, among them Q5 AO3401A, U4 TPS54302, U5 LM393APWR

Commit message: fix: add missing LCSC part numbers
Parts:
- R12: LCSC (none) -> C25755
- R14: LCSC (none) -> C25765
- R15: LCSC (none) -> C25792
- R16: value 13k -> 20k; LCSC (none) -> C25765
- R17: LCSC (none) -> C25744
- R18: value 22k -> 33k; LCSC (none) -> C25779
- R26: LCSC (none) -> C26083
Changed lines of the file:
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@@
       (effects (font (size 1.27 1.27)) hide)
     )
-    (property "LCSC" "" (id 4) (at 135.89 93.98 0)
+    (property "LCSC" "C25744" (id 4) (at 135.89 93.98 0)
       (effects (font (size 1.27 1.27)) hide)
     )
@@
       (effects (font (size 1.27 1.27)) hide)
     )
+    (property "LCSC" "C26083" (id 4) (at 120.65 97.79 0)
+      (effects (font (size 1.27 1.27)) hide)
+    )
     (pin "1")
     (pin "2")
@@
       (effects (font (size 1.27 1.27)) hide)
     )
-    (property "LCSC" "" (id 4) (at 157.48 43.18 0)
+    (property "LCSC" "C25755" (id 4) (at 157.48 43.18 0)
       (effects (font (size 1.27 1.27)) hide)
     )
@@
       (effects (font (size 1.27 1.27)) (justify left))
     )
-    (property "Value" "13k" (id 1) (at 106.9086 93.1422 0)
+    (property "Value" "20k" (id 1) (at 106.9086 93.1422 0)
       (effects (font (size 1.27 1.27)) (justify left))
     )
@@
       (effects (font (size 1.27 1.27)) hide)
     )
-    (property "LCSC" "" (id 4) (at 105.41 91.44 0)
+    (property "LCSC" "C25765" (id 4) (at 105.41 91.44 0)
       (effects (font (size 1.27 1.27)) hide)
     )
@@
       (effects (font (size 1.27 1.27)) (justify left))
     )
-    (property "Value" "22k" (id 1) (at 106.9086 113.4622 0)
+    (property "Value" "33k" (id 1) (at 106.9086 113.4622 0)
       (effects (font (size 1.27 1.27)) (justify left))
     )
@@
       (effects (font (size 1.27 1.27)) hide)
     )
-    (property "LCSC" "" (id 4) (at 105.41 111.76 0)
+    (property "LCSC" "C25779" (id 4) (at 105.41 111.76 0)
       (effects (font (size 1.27 1.27)) hide)
     )
@@
       (effects (font (size 1.27 1.27)) hide)
     )
-    (property "LCSC" "" (id 4) (at 128.27 86.36 0)
+    (property "LCSC" "C25792" (id 4) (at 128.27 86.36 0)
       (effects (font (size 1.27 1.27)) hide)
     )
@@
       (effects (font (size 1.27 1.27)) hide)
     )
-    (property "LCSC" "" (id 4) (at 157.48 53.34 0)
-      (effects (font (size 1.27 1.27)) hide)
-    )
+    (property "LCSC" "C25765" (id 4) (at 157.48 53.34 0)
+      (effects (font (size 1.27 1.27)) hide)
+    )
